File: KiCad files/version1.kicad_sch (KiCad schematic)
At the start: 24 parts, among them J2 AVR-ISP-6, J3 Conn_01x02_Pin, M1 Motor, M2 Motor, Q1 FDN337N, Q2 FDN337N, SW2 SW_DPDT_x2, U1 TP4056-42-ESOP8, U2 ATtiny13A-SS

Commit message: Update
Other:
- note added: "ATtiny13A Microcontroller Unit"
- note added: "Charging Unit"
- note added: "LI sensors unit"
- note added: "Motor1 driver unit"
- note added: "Motor2 driver unit"
- note added: "Programming connector"
- note removed: "ATtiny 13 MCU unit"
- note removed: "Charg Unit"
- note removed: "ISP connector"
- note removed: "LDR unit"
- note removed: "Motor1"
- note removed: "Motor2"
Changed lines of the file:
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@@
 		)
 	)
-	(text "ISP connector\n"
+	(text "Programming connector\n"
 		(exclude_from_sim no)
-		(at 223.52 82.55 0)
+		(at 196.088 85.852 0)
 		(effects
 			(font
@@
 		)
 	)
-	(text "Charg Unit"
+	(text "Charging Unit"
 		(exclude_from_sim no)
-		(at 15.24 87.63 0)
+		(at 16.002 86.868 0)
 		(effects
 			(font
@@
 		)
 	)
-	(text "Motor2\n"
+	(text "Motor2 driver unit\n"
 		(exclude_from_sim no)
-		(at 230.886 158.242 0)
+		(at 220.218 161.036 0)
 		(effects
 			(font
@@
 		)
 	)
-	(text "ATtiny 13 MCU unit\n"
+	(text "ATtiny13A Microcontroller Unit\n\n"
 		(exclude_from_sim no)
-		(at 124.46 85.09 0)
+		(at 107.95 90.17 0)
 		(effects
 			(font
@@
 		)
 	)
-	(text "LDR unit"
+	(text "LI sensors unit"
 		(exclude_from_sim no)
-		(at 49.53 162.56 0)
+		(at 46.99 162.814 0)
 		(effects
 			(font
@@
 		)
 	)
-	(text "Motor1\n"
+	(text "Motor1 driver unit\n\n"
 		(exclude_from_sim no)
-		(at 136.652 160.528 0)
+		(at 127.254 165.354 0)
 		(effects
 			(font

Commit message: updated files
Other:
- note added: "ATtiny13A Microcontroller"
- note added: "Battery"
- note added: "Battery charging circuit"
- note added: "Charging pins"
- note added: "Light intensity sensors"
- note added: "Motor driver circuit 1"
- note added: "Motor driver circuit 2"
- note added: "Programming connector pins"
- note added: "Slide switch"
- note removed: "ATtiny13A Microcontroller Unit"
- note removed: "Battery Unit"
- note removed: "Charging Module"
- note removed: "Charging Pins"
- note removed: "Charging Unit"
- note removed: "LI sensors unit"
- note removed: "Motor1 driver unit"
- note removed: "Motor2 driver unit"
- note removed: "Programming connector"
- note removed: "SlideSwitch"
- moved on the sheet: D1, D2, L1, L2, R1, R10, R2, R3, R8, R9
